File: Rp2040 wearable dev boards w wireless.kicad_sch (KiCad schematic)
At the start: 39 parts

Commit message: started work on adc
Parts:
- added U?: ADS7830, Package_SO:TSSOP-16_4.4x5mm_P0.65mm, symbol Analog_DAC:ADS7830
Connections:
- net External ADC SDA / GPIO 20: now reaches U?.36 (GPIO24)
- net External ADC SCL / GPIO 21: now reaches U?.37 (GPIO25)
- net ADC 1: now reaches U?.38 (GPIO26_ADC0)
- net ADC 2: now reaches U?.39 (GPIO27_ADC1)
- net ADC 3: now reaches U?.40 (GPIO28_ADC2)
- net ADC 4: now reaches U?.41 (GPIO29_ADC3)
Other:
- note added: "I/O and Peripherals)"
- note removed: "I/O and Peripherals"
Changed lines of the file:
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@@
+    (stroke (width 0) (type default) (color 0 0 0 0))
+  )
+  (wire (pts (xy 184.15 242.57) (xy 194.31 242.57))
     (stroke (width 0) (type default) (color 0 0 0 0))
   )
@@
     (stroke (width 0) (type default) (color 0 0 0 0))
   )
+  (wire (pts (xy 184.15 257.81) (xy 194.31 257.81))
+    (stroke (width 0) (type default) (color 0 0 0 0))
+  )
   (wire (pts (xy 307.34 223.52) (xy 307.34 229.87))
     (stroke (width 0) (type default) (color 0 0 0 0))
@@
     (stroke (width 0) (type default) (color 0 0 0 0))
   )
+  (wire (pts (xy 184.15 250.19) (xy 194.31 250.19))
+    (stroke (width 0) (type default) (color 0 0 0 0))
+  )
   (wire (pts (xy 49.53 39.37) (xy 49.53 41.91))
     (stroke (width 0) (type default) (color 0 0 0 0))
@@
     (stroke (width 0) (type default) (color 0 0 0 0))
   )
+  (wire (pts (xy 184.15 252.73) (xy 194.31 252.73))
+    (stroke (width 0) (type default) (color 0 0 0 0))
+  )
   (wire (pts (xy 86.36 116.84) (xy 86.36 120.65))
     (stroke (width 0) (type default) (color 0 0 0 0))
@@
     (stroke (width 0) (type default) (color 0 0 0 0))
   )
+  (wire (pts (xy 184.15 245.11) (xy 194.31 245.11))
+    (stroke (width 0) (type default) (color 0 0 0 0))
+  )
   (wire (pts (xy 184.15 234.95) (xy 194.31 234.95))
     (stroke (width 0) (type default) (color 0 0 0 0))
@@
   )
   (wire (pts (xy 58.42 31.75) (xy 58.42 35.56))
+    (stroke (width 0) (type default) (color 0 0 0 0))
+  )
+  (wire (pts (xy 184.15 255.27) (xy 194.31 255.27))
     (stroke (width 0) (type default) (color 0 0 0 0))
   )
@@
     (effects (font (size 1.27 1.27)) (justify left bottom))
   )
-  (text "I/O and Peripherals" (at 167.64 15.24 0)
+  (text "I/O and Peripherals)" (at 167.64 15.24 0)
     (effects (font (size 1.27 1.27)) (justify left bottom))
   )
@@
     (effects (font (size 1.27 1.27)) (justify right bottom))
   )
+  (label "ADC 1" (at 194.31 250.19 180)
+    (effects (font (size 1.27 1.27)) (justify right bottom))
+  )
   (label "MISO" (at 316.23 209.55 180)
     (effects (font (size 1.27 1.27)) (justify right bottom))
@@
     (effects (font (size 1.27 1.27)) (justify right bottom))
   )
+  (label "ADC 4" (at 194.31 257.81 180)
+    (effects (font (size 1.27 1.27)) (justify right bottom))
+  )
   (label "USB-" (at 93.98 40.64 0)
     (effects (font (size 1.27 1.27)) (justify left bottom))
@@
   )
   (label "Vmain" (at 152.4 114.3 0)
+    (effects (font (size 1.27 1.27)) (justify left bottom))
+  )
+  (label "ADC 2" (at 194.31 252.73 180)
+    (effects (font (size 1.27 1.27)) (justify right bottom))
+  )
+  (label "ADC 3" (at 194.31 255.27 180)
+    (effects (font (size 1.27 1.27)) (justify right bottom))
+  )
+  (label "External ADC SDA {slash} GPIO 20" (at 194.31 242.57 0)
+    (effects (font (size 1.27 1.27)) (justify left bottom))
+  )
+  (label "External ADC SCL {slash} GPIO 21" (at 194.31 245.11 0)
     (effects (font (size 1.27 1.27)) (justify left bottom))
   )
@@
     )
     (pin "1")
+  )
+  (symbol (lib_id "Analog_DAC:ADS7830") (at 189.23 43.18 0) (mirror y) (unit 1)
+    (in_bom yes) (on_board yes) (fields_autoplaced)
+    (property "Reference" "U?" (id 0) (at 189.7506 25.4 0)
+      (effects (font (size 1.27 1.27)) (justify right))
+    )
+    (property "Value" "ADS7830" (id 1) (at 189.7506 27.94 0)
+      (effects (font (size 1.27 1.27)) (justify right))
+    )
+    (property "Footprint" "Package_SO:TSSOP-16_4.4x5mm_P0.65mm" (id 2) (at 186.69 60.96 0)
+      (effects (font (size 1.27 1.27) italic) hide)
+    )
+    (property "Datasheet" "http://www.ti.com/lit/ds/symlink/ads7830.pdf" (id 3) (at 184.15 54.61 0)
+      (effects (font (size 1.27 1.27)) hide)
+    )
+    (pin "1")
+    (pin "10")
+    (pin "11")
+    (pin "12")
+    (pin "13")
+    (pin "14")
+    (pin "15")
+    (pin "16")
+    (pin "2")
+    (pin "3")
+    (pin "4")
+    (pin "5")
+    (pin "6")
+    (pin "7")
+    (pin "8")
+    (pin "9")
   )
   (symbol (lib_id "power:GND") (at 314.96 241.3 0) (unit 1)
@@
       (reference "U?") (unit 1) (value "LTH7R") (footprint "Package_TO_SOT_SMD:SOT-23-5")
     )
+    (path "/8cb7f4bd-c777-4d24-a1be-b9a8ac248327"
+      (reference "U?") (unit 1) (value "ADS7830") (footprint "Package_SO:TSSOP-16_4.4x5mm_P0.65mm")
+    )
     (path "/ccdd1266-dc76-406c-a364-69f8ab51981c"

Commit message: yeh, stuff happened finished rp2040 pinout, added the IMU that is going to be used, created a set of solder pads (x21) for the GPIO
Parts:
- removed C? (x2): C, symbol Device:C
- removed R?: R, symbol Device:R
- removed Y?: Crystal, symbol Device:Crystal
- added C? (x9): 100n, symbol Device:C
- added C? (x2): 1u, symbol Device:C
- added C? (x2): 27p, symbol Device:C
- added C?: C, symbol Device:C
- added J?: Conn_01x21, edge tabs:Edge solder pads x21, symbol Connector_Generic:Conn_01x21
- added R?: 1K, symbol Device:R
- added R? (x2): 27.4, symbol Device:R
- added R?: 1k, symbol Device:R
- added SW?: SW_Push, symbol Switch:SW_Push
- added U?: MPU-6050, Sensor_Motion:InvenSense_QFN-24_4x4mm_P0.5mm, symbol Sensor_Motion:MPU-6050
- added Y?: ABLS-12.000MHZ-B4-T, symbol Device:Crystal
Connections:
- net +3V3 is gone; now on net +3.3V: C?.1, C?.1, C?.1, IC?.15 (VDD_2), IC?.18 (VDD_3), IC?.7 (VDD_1), U?.2 (VO)
- net External ADC SCL / GPIO 21: now also J?.21 (Pin_21)
- net External ADC SDA / GPIO 20: now also J?.20 (Pin_20)
- net GND: now also U?.19 (TESTEN), U?.4 (GND), U?.57 (GND), C?.2, C?.2, C?.2, C?.2, C?.2, C?.2, C?.2, C?.2, C?.2, C?.2, C?.2, C?.2, C?.2, C?.2, SW?.1
- net USB+: now also R?.1
- net USB-: now also R?.1
- net +3.3V: now reaches U?.1 (IOVDD), U?.10 (IOVDD), U?.22 (IOVDD), U?.33 (IOVDD), U?.42 (IOVDD), U?.49 (IOVDD)
- net +3.3V: now also U?.43 (ADC_AVDD), U?.44 (VREG_IN), U?.48 (USB_VDD), U?.8 (VCC), C?.1, C?.1, C?.1, C?.1, C?.1, C?.1, C?.1, C?.1, C?.1
- net GPIO 8: now reaches U?.11 (GPIO8)
- net GPIO 8: now also J?.8 (Pin_8)
- net GPIO 9: now reaches U?.12 (GPIO9)
- net GPIO 9: now also J?.9 (Pin_9)
- net GPIO 10: now reaches U?.13 (GPIO10)
- net GPIO 10: now also J?.10 (Pin_10)
- net GPIO 11: now reaches U?.14 (GPIO11)
- net GPIO 11: now also J?.11 (Pin_11)
- net GPIO 12: now reaches U?.15 (GPIO12)
- net GPIO 12: now also J?.12 (Pin_12)
- net GPIO 13: now reaches U?.16 (GPIO13)
- net GPIO 13: now also J?.13 (Pin_13)
- net GPIO 14: now reaches U?.17 (GPIO14)
- net GPIO 14: now also J?.14 (Pin_14)
- net GPIO 15: now reaches U?.18 (GPIO15)
- net GPIO 15: now also J?.15 (Pin_15)
- net GPIO 0: now reaches U?.2 (GPIO0)
- net GPIO 0: now also J?.1 (Pin_1)
- net XIN: now reaches U?.20 (XIN)
- net XIN: now also C?.1, Y?.2
- net XOUT: now reaches U?.21 (XOUT)
- net XOUT: now also R?.2
- net +1V1: now reaches U?.23 (DVDD), U?.50 (DVDD)
- net +1V1: now also U?.45 (VREG_VOUT), C?.1, C?.1, C?.1
- net run: now reaches U?.26 (RUN)
- net GPIO 16: now reaches U?.27 (GPIO16)
- net GPIO 16: now also J?.16 (Pin_16)
- net GPIO 17: now reaches U?.28 (GPIO17)
- net GPIO 17: now also J?.17 (Pin_17)
- net IMU SDA / GPIO 18: now reaches U?.29 (GPIO18)
- net IMU SDA / GPIO 18: now also J?.18 (Pin_18)
- net GPIO 1: now reaches U?.3 (GPIO1)
- net GPIO 1: now also J?.2 (Pin_2)
- net IMU SCL / GPIO 19: now reaches U?.30 (GPIO19)
- net IMU SCL / GPIO 19: now also J?.19 (Pin_19)
- net GPIO 2: now reaches U?.4 (GPIO2)
- net at U?.46 (USB_DM): now also R?.2
- net at U?.47 (USB_DP): now also R?.2
- net GPIO 3: now reaches U?.5 (GPIO3)
- net GPIO 3: now also J?.3 (Pin_3)
- net QSPI_SD3: now reaches U?.51 (QSPI_SD3), U?.7 (IO3)
- net QSPI_SCLK: now reaches U?.52 (QSPI_SCLK)
- net QSPI_SCLK: now also U?.6 (CLK)
- net QSPI_SD0: now reaches U?.5 (DI(IO0)), U?.53 (QSPI_SD0)
- net QSPI_SD2: now reaches U?.3 (IO2), U?.54 (QSPI_SD2)
- net QSPI_SD1: now reaches U?.2 (DO(IO1)), U?.55 (QSPI_SD1)
- net QSPI_SS: now reaches U?.56 (QSPI_SS)
- net QSPI_SS: now also U?.1 (~{CS}), R?.2
- net GPIO 4: now reaches U?.6 (GPIO4)
- net GPIO 4: now also J?.4 (Pin_4)
- net GPIO 5: now reaches U?.7 (GPIO5)
- net GPIO 5: now also J?.5 (Pin_5)
- net GPIO 6: now reaches U?.8 (GPIO6)
- net GPIO 6: now also J?.6 (Pin_6)
- net GPIO 7: now reaches U?.9 (GPIO7)
- net GPIO 7: now also J?.7 (Pin_7)
- new net XOUTC: C?.1, R?.1, Y?.1
- new net ~{USB BOOT}: R?.1, SW?.2
Other:
- note added: "6-axis gyro/accel (3 rot, 3 lin)"
- note added: "extended ADC"
- note added: "idk looks like a bunch of pins have been hidden"
- note added: "note, external ADC takes I^{2}C bus one Radio takes SPI bus one imu takes I^{2}C bus two I will pin them out"
- note added: "one cap per power pin 1uf caps are for pin's 44 and 45"
- note added: "these names on the lines help with routing later"
- note added: "this is the boot button, I cant understand what they are saying in the data sheet abt it"
- moved on the sheet: U?

Commit message: finnished preiferals added names and pads
Parts:
- removed U?: MPU-6050, Sensor_Motion:InvenSense_QFN-24_4x4mm_P0.5mm, symbol Sensor_Motion:MPU-6050
- removed Y?: Crystal, symbol Device:Crystal
- added C11, C19: 10u, Capacitor_SMD:C_01005_0402Metric, symbol Device:C_Polarized_Small
- added C12, C23: 0.1u, Capacitor_SMD:C_01005_0402Metric, symbol Device:C
- added C21: 0.2u, Capacitor_SMD:C_01005_0402Metric, symbol Device:C
- added C22: 10n, Capacitor_SMD:C_01005_0402Metric, symbol Device:C
- added J4: Conn_01x18, Connector_PinSocket_2.54mm:PinSocket_1x18_P2.54mm_Horizontal, symbol Connector_Generic:Conn_01x18
- added R10: 5, Resistor_SMD:R_0402_1005Metric, symbol Device:R
- added R11, R12: 2K, Resistor_SMD:R_0402_1005Metric, symbol Device:R
- added U7: MPU-6500, QFN24_3X3X0P9_IVS, symbol MPU-6500:MPU-6500
- added Y2: ECS-160-9-42-CKM-TR, ECS-160-9-42-CKM-TR:XTAL_ECS-160-9-42-CKM-TR, symbol Device:Crystal_GND24
- AE1: renamed from AE?; footprint (none) -> coaxial conn:MURATA_MM8030-2610RJ3
- C1, C10, C13, C14, C15, C16, C17, C18, C2, C20, C26, C27, C28, C29, C30, C31, C32, C4, C5, C6, C7, C8, C9: renamed from C?; footprint (none) -> Capacitor_SMD:C_01005_0402Metric
- C24, C25: renamed from C?; value C -> 14p; footprint (none) -> Capacitor_SMD:C_01005_0402Metric
- C3: renamed from C?; value C -> 100n; footprint (none) -> Capacitor_SMD:C_01005_0402Metric
- J2: renamed from J?; value USB_C_Receptacle -> UJ31-CH-31-SMT-TR; footprint (none) -> usb-c footprint:CUI_UJ31-CH-31-SMT-TR
- L1, L2, L3: renamed from L?; footprint (none) -> Inductor_SMD:L_0402_1005Metric
- R1, R14, R2, R4, R6, R7: renamed from R?; footprint (none) -> Resistor_SMD:R_0402_1005Metric
- R13: renamed from R?; value R -> 1M; footprint (none) -> Resistor_SMD:R_0402_1005Metric
- SW1: renamed from SW?; value SW_Push -> B3U-1100P; footprint (none) -> Button_Switch_SMD:SW_SPST_B3U-1100P
- Y1: renamed from Y?; footprint (none) -> ABLS-12:ABLS-12.000MHZ-B4-T
- gave numbers to parts that had none: 16
Connections:
- net +3.3V: now also C19.1, C21.1, C22.1, J4.15 (Pin_15), J4.2 (Pin_2), R10.2, R11.1, R12.1, U7.13 (VDD), U7.8 (VDDIO)
- net ADC 1: now also J4.11 (Pin_11)
- net ADC 2: now also J4.12 (Pin_12)
- net ADC 3: now also J4.13 (Pin_13)
- net ADC 4: now also J4.14 (Pin_14)
- net External ADC SCL / GPIO 21: now also U6.14 (SCL), U6.15 (SDA), R11.2
- net External ADC SDA / GPIO 20: now also R12.2
- net GND: now also U6.12 (A0), U6.13 (A1), U6.9 (GND), C11.2, C12.2, C19.2, C21.2, C22.2, C23.2, J4.17 (Pin_17), J4.18 (Pin_18), U7.11 (FSYNC), U7.12 (INT), U7.18 (GND), U7.20 (RESV), U7.22 (nCS), U7.9 (SDO/ADO), Y2.2, Y2.4
- net IMU SCL / GPIO 19: now also U7.23 (SCL/SCLK)
- net IMU SDA / GPIO 18: now also U7.24 (SDA/SDI)
- net VBUS: now also J4.1 (Pin_1), J4.16 (Pin_16)
- net VDD_PA: now reaches C29.1, C30.1, IC1.11 (VDD_PA), L3.2
- net XC2: now reaches C25.1, IC1.9 (XC2), R13.2
- net XC2: now also Y2.3
- net XC1: now reaches C24.1, IC1.10 (XC1), R13.1
- net XC1: now also Y2.1
- net ANT 2: now reaches IC1.13 (ANT2), L1.2, L3.1
- net ANT 1: now reaches IC1.12 (ANT1), L1.1, L2.1
- net ACH0: now reaches U6.1 (CH0)
- net ACH0: now also J4.3 (Pin_3)
- net refin: now reaches U6.10 (REFin/REFout)
- net refin: now also C12.1
- net COM: now reaches U6.11 (COM)
- net COM: now also J4.10 (Pin_10)
- net at U6.16 (VDD): now also C11.1, R10.1
- net ACH1: now reaches U6.2 (CH1)
- net ACH1: now also J4.4 (Pin_4)
- net ACH2: now reaches U6.3 (CH2)
- net ACH2: now also J4.5 (Pin_5)
- net ACH3: now reaches U6.4 (CH3)
- net ACH3: now also J4.6 (Pin_6)
- net ACH4: now reaches U6.5 (CH4)
- net ACH5: now reaches U6.6 (CH5)
- net ACH5: now also J4.7 (Pin_7)
- net ACH6: now reaches U6.7 (CH6)
- net ACH6: now also J4.8 (Pin_8)
- net ACH7: now reaches U6.8 (CH7)
- net ACH7: now also J4.9 (Pin_9)
- new net: C23.1, U7.10 (REGOUT)
- new net AUX_CL: U7.7 (AUX_CL)
- new net AUX_DA: U7.21 (AUX_DA)
Other:
- moved on the sheet: U6

Commit message: finished schematic v.1 about to start routing
Parts:
- removed J3: Conn_01x21, edge tabs:Edge solder pads x21, symbol Connector_Generic:Conn_01x21
- added D3: LED_YELLOW, LED_SMD:LED_0603_1608Metric, symbol Device:LED
- added D4: LED_GREEN, LED_SMD:LED_0603_1608Metric, symbol Device:LED
- added J?: Conn_01x22, symbol Connector_Generic:Conn_01x22
- added R15, R16, R17: 2K, Resistor_SMD:R_0402_1005Metric, symbol Device:R
- D1: value LED -> LED_BLUE
- U3: footprint DQA0010A -> TPD4E02B04QDQARQ1:TPD4E02B04QDQARQ1
- U7: footprint QFN24_3X3X0P9_IVS -> MPU-6500:MPU-6500
Connections:
- net +3.3V: now also R16.1, R17.1
- net External ADC SCL / GPIO 21: now also J?.21 (Pin_21)
- net External ADC SDA / GPIO 20: now also J?.20 (Pin_20)
- net GND: now also D3.1 (K), D4.1 (K); no longer SW1.1
- net GPIO 0: now also J?.1 (Pin_1), R15.1
- net GPIO 1: now also J?.2 (Pin_2)
- net GPIO 10: now also J?.10 (Pin_10)
- net GPIO 11: now also J?.11 (Pin_11)
- net GPIO 12: now also J?.12 (Pin_12)
- net GPIO 13: now also J?.13 (Pin_13)
- net GPIO 14: now also J?.14 (Pin_14)
- net GPIO 15: now also J?.15 (Pin_15)
- net GPIO 16: now also J?.16 (Pin_16)
- net GPIO 17: now also J?.17 (Pin_17)
- net GPIO 3: now also J?.3 (Pin_3)
- net GPIO 4: now also J?.4 (Pin_4)
- net GPIO 5: now also J?.5 (Pin_5)
- net GPIO 6: now also J?.6 (Pin_6)
- net GPIO 7: now also J?.7 (Pin_7)
- net GPIO 8: now also J?.8 (Pin_8)
- net GPIO 9: now also J?.9 (Pin_9)
- net IMU SCL / GPIO 19: now also J?.19 (Pin_19), R16.2
- net IMU SDA / GPIO 18: now also J?.18 (Pin_18), R17.2
- net SWCLK: now reaches U5.24 (SWCLK)
- net SWD: now reaches U5.25 (SWD)
- net run renamed RUN
- net RUN: now also J?.22 (Pin_22)
- new net: D4.2 (A), R15.2
- new net: D3.2 (A), SW1.1
Other:
- note added: "a second version can have the amp on here"
- moved on the sheet: C19, R11, R12

Commit message: finished schematic started pcb design, will need to review the power section.
Parts:
- removed J4: Conn_01x18, Connector_PinSocket_2.54mm:PinSocket_1x18_P2.54mm_Horizontal, symbol Connector_Generic:Conn_01x18
- removed J?: Conn_01x22, symbol Connector_Generic:Conn_01x22
- added J3: 3040-40-00, Connector_IDC:IDC-Header_2x20_P2.54mm_Vertical, symbol Connector_Generic:Conn_01x40
- added J4: serial wire debug port, Connector_JST:JST_PH_S2B-PH-SM4-TB_1x02-1MP_P2.00mm_Horizontal, symbol Connector_Generic:Conn_01x02
- added R18: 0, Resistor_SMD:R_0402_1005Metric, symbol Device:R
- added TP1: 3.3v test point, TestPoint:TestPoint_Pad_D2.0mm, symbol Connector:TestPoint
- added TP2: ground test point, TestPoint:TestPoint_Pad_D2.0mm, symbol Connector:TestPoint
- added TP3: rf test point, TestPoint:TestPoint_Pad_D2.0mm, symbol Connector:TestPoint
- C11, C19: footprint Capacitor_SMD:C_01005_0402Metric -> Capacitor_SMD:CP_Elec_5x5.3
- U1: value LTH7R -> MCP73831T-4ADI/OT
Connections:
- net +3.3V: now also J3.35 (Pin_35), J3.36 (Pin_36), J3.37 (Pin_37), R18.2; no longer C9.1, U4.2 (VO)
- net ACH0: now also J3.23 (Pin_23)
- net ACH1: now also J3.24 (Pin_24)
- net ACH2: now also J3.25 (Pin_25)
- net ACH3: now also J3.26 (Pin_26)
- net ACH5: now also J3.27 (Pin_27)
- net ACH6: now also J3.28 (Pin_28)
- net ACH7: now also J3.29 (Pin_29)
- net ADC 1: now also J3.31 (Pin_31)
- net ADC 2: now also J3.32 (Pin_32)
- net ADC 3: now also J3.33 (Pin_33)
- net ADC 4: now also J3.34 (Pin_34)
- net COM: now also J3.30 (Pin_30)
- net External ADC SCL / GPIO 21: now also J3.21 (Pin_21)
- net External ADC SDA / GPIO 20: now also J3.20 (Pin_20)
- net GND: now also J3.38 (Pin_38), J3.39 (Pin_39), J3.40 (Pin_40), TP2.1
- net GPIO 0: now also J3.1 (Pin_1)
- net GPIO 1: now also J3.2 (Pin_2)
- net GPIO 10: now also J3.10 (Pin_10)
- net GPIO 11: now also J3.11 (Pin_11)
- net GPIO 12: now also J3.12 (Pin_12)
- net GPIO 13: now also J3.13 (Pin_13)
- net GPIO 14: now also J3.14 (Pin_14)
- net GPIO 15: now also J3.15 (Pin_15)
- net GPIO 16: now also J3.16 (Pin_16)
- net GPIO 17: now also J3.17 (Pin_17)
- net GPIO 3: now also J3.3 (Pin_3)
- net GPIO 4: now also J3.4 (Pin_4)
- net GPIO 5: now also J3.5 (Pin_5)
- net GPIO 6: now also J3.6 (Pin_6)
- net GPIO 7: now also J3.7 (Pin_7)
- net GPIO 8: now also J3.8 (Pin_8)
- net GPIO 9: now also J3.9 (Pin_9)
- net IMU SCL / GPIO 19: now also J3.19 (Pin_19)
- net IMU SDA / GPIO 18: now also J3.18 (Pin_18)
- net RUN: now also J3.22 (Pin_22)
- net SWCLK: now also J4.1 (Pin_1)
- net SWD: now also J4.2 (Pin_2)
- net at AE1.1 (A), C31.2, C32.1: now also TP3.1
- new net: C9.1, R18.1, TP1.1, U4.2 (VO)
Other:
- note added: "only connect this after confirming it works, yes its a 0 ohm resistor"
- note added: "use part number 1454-1000570038-DS-ND for wire connection"
- moved on the sheet: C5, C9, D1, D2, J1, Q1, R2, R3, R5, U1, U4

Commit message: mmmmmmmmmmm change log.exe
Parts:
- removed AE1: Antenna, coaxial conn:MURATA_MM8030-2610RJ3, symbol Device:Antenna
- removed J3: 3040-40-00, Connector_IDC:IDC-Header_2x20_P2.54mm_Vertical, symbol Connector_Generic:Conn_01x40
- removed J4: serial wire debug port, Connector_JST:JST_PH_S2B-PH-SM4-TB_1x02-1MP_P2.00mm_Horizontal, symbol Connector_Generic:Conn_01x02
- added J3, J4: Conn_01x20, Connector_FFC-FPC:TE_2-84952-0_1x20-1MP_P1.0mm_Horizontal, symbol Connector_Generic:Conn_01x20
- added J5: Conn_01x04, Connector_PinSocket_2.54mm:PinSocket_2x02_P2.54mm_Horizontal, symbol Connector_Generic:Conn_01x04
- added J6: EMPCB.SMAFSTJ.B.HT, TAOGLAS_EMPCB.SMAFSTJ.B.HT, symbol EMPCB.SMAFSTJ.B.HT:EMPCB.SMAFSTJ.B.HT
- added SW2: power Switch, Connector_JST:JST_PH_S2B-PH-SM4-TB_1x02-1MP_P2.00mm_Horizontal, symbol Switch:SW_SPST
- IC1: footprint QFN50P400X400X95-21N-D -> LIB_NRF24L01P-R7:QFN50P400X400X95-21N-D
- U3: footprint TPD4E02B04QDQARQ1:TPD4E02B04QDQARQ1 -> LIB_TPD4E02B04QDQARQ1:TPD4E02B04QDQARQ1
- U4: footprint Package_TO_SOT_SMD:TO-252-2 -> Package_TO_SOT_SMD:SOT-223
Connections:
- net ACH0: now also J4.4 (Pin_4)
- net ACH1: now also J4.5 (Pin_5)
- net ACH2: now also J4.6 (Pin_6)
- net ACH3: now also J4.7 (Pin_7)
- net ACH5: now also J4.8 (Pin_8)
- net ACH6: now also J4.9 (Pin_9)
- net ACH7: now also J4.10 (Pin_10)
- net ADC 1: now also J4.12 (Pin_12)
- net ADC 2: now also J4.13 (Pin_13)
- net ADC 3: now also J4.14 (Pin_14)
- net ADC 4: now also J4.15 (Pin_15)
- net AUX_CL: now also J4.18 (Pin_18)
- net AUX_DA: now also J4.17 (Pin_17)
- net COM: now also J4.11 (Pin_11)
- net External ADC SCL / GPIO 21: now also J5.4 (Pin_4)
- net External ADC SDA / GPIO 20: now also J5.3 (Pin_3)
- net GND: now also J3.20 (Pin_20), J4.20 (Pin_20), J6.SH1, J6.SH2, J6.SH3, J6.SH4
- net GPIO 0: now also J3.1 (Pin_1), J4.1 (Pin_1)
- net GPIO 1: now also J3.2 (Pin_2)
- net GPIO 10: now also J3.10 (Pin_10)
- net GPIO 11: now also J3.11 (Pin_11)
- net GPIO 12: now also J3.12 (Pin_12)
- net GPIO 13: now also J3.13 (Pin_13)
- net GPIO 14: now also J3.14 (Pin_14)
- net GPIO 15: now also J3.15 (Pin_15)
- net GPIO 16: now also J4.2 (Pin_2)
- net GPIO 17: now also J4.3 (Pin_3)
- net GPIO 3: now also J3.3 (Pin_3)
- net GPIO 4: now also J3.4 (Pin_4)
- net GPIO 5: now also J3.5 (Pin_5)
- net GPIO 6: now also J3.6 (Pin_6)
- net GPIO 7: now also J3.7 (Pin_7)
- net GPIO 8: now also J3.8 (Pin_8)
- net GPIO 9: now also J3.9 (Pin_9)
- net IMU SCL / GPIO 19: now also J5.2 (Pin_2)
- net IMU SDA / GPIO 18: now also J5.1 (Pin_1)
- net RUN: now also J3.16 (Pin_16), J4.16 (Pin_16)
- net SWCLK: now also J3.17 (Pin_17)
- net SWD: now also J3.18 (Pin_18)
- net USB+: now also J2.A7 (D-), J2.B7 (D-); no longer J2.A6 (D+), J2.B6 (D+)
- net USB-: now also J2.A6 (D+), J2.B6 (D+); no longer J2.A7 (D-), J2.B7 (D-)
- net VO: now reaches C9.1, R18.1, TP1.1, U4.2 (VO)
- net VI: now reaches C5.1, D2.1 (K), Q1.2 (S), U4.3 (VI)
- net CC2: now reaches R9.1, U3.1 (D1+), U3.10 (NC)
- net CC2: now also J2.B5 (CC2); no longer J2.A5 (CC1)
- net CC1: now reaches R8.1, U3.2 (D1-), U3.9 (NC)
- net CC1: now also J2.A5 (CC1); no longer J2.B5 (CC2)
- net LED_GREEN: now reaches D4.2 (A), R15.2
- net STAT: now reaches R3.2, U1.1 (STAT)
- net PROG: now reaches R2.1, U1.5 (PROG)
- net ADC VDD: now reaches C11.1, R10.1, U6.16 (VDD)
- net LED_BLUE: now reaches D1.1 (K), R3.1
- net SW1 : now reaches D3.2 (A), SW1.1
- net Antenna: now reaches C31.2, C32.1, TP3.1
- net Antenna: now also J6.1
- net L2-C31: now reaches C31.1, L2.2
- net DVDD_RADIO: now reaches C28.1, IC1.19 (DVDD)
- net REGOUT: now reaches C23.1, U7.10 (REGOUT)
- net IREF: now reaches IC1.16 (IREF), R14.2
- net USB_R-: now reaches R7.2, U5.46 (USB_DM)
- net USB_R+: now reaches R6.2, U5.47 (USB_DP)
- net +1V1 renamed DVDD_RP2040
- net +3.3V renamed Vmain
- net Vmain: now also J3.19 (Pin_19), J4.19 (Pin_19), SW2.2 (B); no longer R18.2
- net refin renamed REFin/REFout
- new net R18-Power_on: R18.2, SW2.1 (A)
Other:
- note added: "GPIO 0-15 are used as wrist mounted pins, read the data sheet to see what can and cant be done with them"
- note added: "GPIO 16+17 are used for UART 0 Rx, Tx this is for an external connect on hand"
- note added: "J3 and J4 are FFC connectors to save space"
- note added: "dont ask, routing becomes easier like this"
- note added: "ok quick explanation, GPIO 0 is a debug led, so both hand and wrist get it wrist cannot use its periferal functions tho"
- note added: "some debug pinouts"
- note added: "to hand mount"
- note added: "to periferals on wrist / near board"
- note removed: "use part number 1454-1000570038-DS-ND for wire connection"
- moved on the sheet: R18
