File: Rp2040 wearable dev boards w wireless.kicad_sch (KiCad schematic)
At the start: 79 parts, among them IC1 NRF24L01P-R7, J1 battery plug, J2 DX07S016JA1R1500, J3 Conn_01x20, J4 Conn_01x20, J6 EMPCB.SMAFSTJ.B.HT, Q1 Si2301, SW1 B3U-1100P, SW2 power Switch, U1 MCP73831T-4ADI/OT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

Commit message: finished
Parts:
- R1: Digikey Part  Number (none) -> 311-1.0KJRCT-ND
- R10: value 5 -> 330; Digikey Part  Number (none) -> 311-330JRCT-ND
- R11, R12, R15, R16, R17, R19, R2: Digikey Part  Number (none) -> YAG2303CT-ND
- R13: Digikey Part  Number (none) -> 311-1.0MJRCT-ND
- R14: Digikey Part  Number (none) -> 311-22.0KLRCT-ND
- R18: Digikey Part  Number (none) -> 311-0.0LRCT-ND
- R3, R4: Digikey Part  Number (none) -> 311-10KJRCT-ND
- R5: Digikey Part  Number (none) -> 13-RC0402FR-13100KLCT-ND
- R6, R7: Digikey Part  Number (none) -> YAG3085CT-ND
- R8, R9: Digikey Part  Number (none) -> 13-RC0402FR-135K1LCT-ND
- SW1: Digikey Part  Number (none) -> SW1021CT-ND
- SW2: Digikey Part  Number (none) -> 455-1749-1-ND
- TP1, TP3: Digikey Part  Number (none) -> n/a
- U1: Digikey Part  Number (none) -> MCP73831T-4ADI/OTCT-ND
- U2: Digikey Part  Number (none) -> W25Q128JVSIMCT-ND
- U3: Digikey Part  Number (none) -> 296-48995-1-ND
- U4: Digikey Part  Number (none) -> NCP1117LPST33T3GOSCT-ND
- U5: Digikey Part  Number (none) -> 2648-SC0914(13)CT-ND
- U6: Digikey Part  Number (none) -> 296-25899-1-ND
- U7: Digikey Part  Number (none) -> 1428-1011-1-ND
- Y1: Digikey Part  Number (none) -> CTX1162CT-ND
- Y2: Digikey Part  Number (none) -> XC1611CT-ND
Changed lines of the file:
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@@
+      (effects (font (size 1.27 1.27)) hide)
+    )
+    (property "Digikey Part  Number" "NCP1117LPST33T3GOSCT-ND" (id 4) (at 121.92 114.3 0)
       (effects (font (size 1.27 1.27)) hide)
     )
@@
       (effects (font (size 1.524 1.524)))
     )
+    (property "Digikey Part  Number" "296-48995-1-ND" (id 4) (at 72.39 41.91 0)
+      (effects (font (size 1.27 1.27)) hide)
+    )
     (pin "1")
     (pin "10")
@@
       (effects (font (size 1.27 1.27)) hide)
     )
+    (property "Digikey Part  Number" "YAG2303CT-ND" (id 4) (at 198.12 181.61 0)
+      (effects (font (size 1.27 1.27)) hide)
+    )
     (pin "1")
     (pin "2")
@@
     )
     (property "Datasheet" "http://ww1.microchip.com/downloads/en/DeviceDoc/20001984g.pdf" (id 3) (at 41.91 119.38 0)
+      (effects (font (size 1.27 1.27)) hide)
+    )
+    (property "Digikey Part  Number" "MCP73831T-4ADI/OTCT-ND" (id 4) (at 45.72 118.11 0)
       (effects (font (size 1.27 1.27)) hide)
     )
@@
       (effects (font (size 1.27 1.27)) hide)
     )
+    (property "Digikey Part  Number" "13-RC0402FR-13100KLCT-ND" (id 4) (at 90.17 139.7 0)
+      (effects (font (size 1.27 1.27)) hide)
+    )
     (pin "1")
     (pin "2")
@@
       (effects (font (size 1.27 1.27)) hide)
     )
+    (property "Digikey Part  Number" "455-1749-1-ND" (id 4) (at 151.13 114.3 0)
+      (effects (font (size 1.27 1.27)) hide)
+    )
     (pin "1")
     (pin "2")
@@
       (effects (font (size 1.27 1.27)) hide)
     )
+    (property "Digikey Part  Number" "YAG2303CT-ND" (id 4) (at 312.42 212.09 0)
+      (effects (font (size 1.27 1.27)) hide)
+    )
     (pin "1")
     (pin "2")
@@
     (in_bom yes) (on_board yes)
     (property "Reference" "R10" (id 0) (at 214.63 19.05 90))
-    (property "Value" "5" (id 1) (at 215.9 21.59 90))
+    (property "Value" "330" (id 1) (at 215.9 21.59 90))
     (property "Footprint" "Resistor_SMD:R_0402_1005Metric" (id 2) (at 215.9 23.368 90)
       (effects (font (size 1.27 1.27)) hide)
     )
     (property "Datasheet" "~" (id 3) (at 215.9 21.59 0)
+      (effects (font (size 1.27 1.27)) hide)
+    )
+    (property "Digikey Part  Number" "311-330JRCT-ND" (id 4) (at 215.9 21.59 0)
       (effects (font (size 1.27 1.27)) hide)
     )
@@
       (effects (font (size 1.27 1.27)) hide)
     )
+    (property "Digikey Part  Number" "311-1.0MJRCT-ND" (id 4) (at 311.15 229.87 0)
+      (effects (font (size 1.27 1.27)) hide)
+    )
     (pin "1")
     (pin "2")
@@
     )
     (property "Datasheet" "~" (id 3) (at 403.86 191.77 0)
+      (effects (font (size 1.27 1.27)) hide)
+    )
+    (property "Digikey Part  Number" "n/a" (id 4) (at 398.78 191.77 0)
       (effects (font (size 1.27 1.27)) hide)
     )
@@
     )
     (property "Datasheet" "~" (id 3) (at 69.85 113.03 0)
+      (effects (font (size 1.27 1.27)) hide)
+    )
+    (property "Digikey Part  Number" "311-10KJRCT-ND " (id 4) (at 69.85 113.03 0)
       (effects (font (size 1.27 1.27)) hide)
     )
@@
       (effects (font (size 1.27 1.27)) hide)
     )
+    (property "Digikey Part  Number" "13-RC0402FR-135K1LCT-ND" (id 4) (at 120.65 43.18 0)
+      (effects (font (size 1.27 1.27)) hide)
+    )
     (pin "1")
     (pin "2")
@@
       (effects (font (size 1.27 1.27)) hide)
     )
+    (property "Digikey Part  Number" "YAG2303CT-ND" (id 4) (at 34.29 125.73 0)
+      (effects (font (size 1.27 1.27)) hide)
+    )
     (pin "1")
     (pin "2")
@@
     )
     (property "Datasheet" "~" (id 3) (at 260.35 233.68 0)
+      (effects (font (size 1.27 1.27)) hide)
+    )
+    (property "Digikey Part  Number" "YAG2303CT-ND" (id 4) (at 260.35 233.68 0)
       (effects (font (size 1.27 1.27)) hide)
     )
@@
       (effects (font (size 1.27 1.27)) hide)
     )
+    (property "Digikey Part  Number" "SW1021CT-ND" (id 4) (at 16.51 213.36 0)
+      (effects (font (size 1.27 1.27)) hide)
+    )
     (pin "1")
     (pin "2")
@@
       (effects (font (size 1.27 1.27)) hide)
     )
+    (property "Digikey Part  Number" "XC1611CT-ND" (id 4) (at 311.15 220.98 0)
+      (effects (font (size 1.27 1.27)) hide)
+    )
     (pin "1")
     (pin "2")
@@
     )
     (property "Datasheet" "http://www.ti.com/lit/ds/symlink/ads7830.pdf" (id 3) (at 204.47 55.88 0)
+      (effects (font (size 1.27 1.27)) hide)
+    )
+    (property "Digikey Part  Number" "296-25899-1-ND" (id 4) (at 209.55 44.45 0)
       (effects (font (size 1.27 1.27)) hide)
     )
@@
       (effects (font (size 1.27 1.27)) hide)
     )
+    (property "Digikey Part  Number" "311-0.0LRCT-ND " (id 4) (at 139.7 114.3 0)
+      (effects (font (size 1.27 1.27)) hide)
+    )
     (pin "1")
     (pin "2")
@@
       (effects (font (size 1.27 1.27)) hide)
     )
+    (property "Digikey Part  Number" "311-1.0KJRCT-ND" (id 4) (at 33.02 208.28 0)
+      (effects (font (size 1.27 1.27)) hide)
+    )
     (pin "1")
     (pin "2")
@@
       (effects (font (size 1.27 1.27)) hide)
     )
+    (property "Digikey Part  Number" "CTX1162CT-ND " (id 4) (at 78.74 242.57 0)
+      (effects (font (size 1.27 1.27)) hide)
+    )
     (pin "1")
     (pin "2")
@@
     (property "Datasheet" "" (id 3) (at 299.72 44.45 0)
       (effects (font (size 1.524 1.524)))
+    )
+    (property "Digikey Part  Number" "1428-1011-1-ND" (id 4) (at 264.16 30.48 0)
+      (effects (font (size 1.27 1.27)) hide)
     )
     (pin "1")
@@
       (effects (font (size 1.27 1.27)) hide)
     )
+    (property "Digikey Part  Number" "YAG2303CT-ND" (id 4) (at 252.73 236.22 0)
+      (effects (font (size 1.27 1.27)) hide)
+    )
     (pin "1")
     (pin "2")
@@
       (effects (font (size 1.27 1.27)) hide)
     )
+    (property "Digikey Part  Number" "YAG3085CT-ND" (id 4) (at 111.76 193.04 0)
+      (effects (font (size 1.27 1.27)) hide)
+    )
     (pin "1")
     (pin "2")
@@
       (effects (font (size 1.27 1.27)) hide)
     )
+    (property "Digikey Part  Number" "13-RC0402FR-135K1LCT-ND" (id 4) (at 128.27 43.18 0)
+      (effects (font (size 1.27 1.27)) hide)
+    )
     (pin "1")
     (pin "2")
@@
     )
     (property "Datasheet" "https://datasheets.raspberrypi.com/rp2040/rp2040-datasheet.pdf" (id 3) (at 158.75 219.71 0)
+      (effects (font (size 1.27 1.27)) hide)
+    )
+    (property "Digikey Part  Number" "2648-SC0914(13)CT-ND" (id 4) (at 158.75 219.71 0)
       (effects (font (size 1.27 1.27)) hide)
     )
@@
       (effects (font (size 1.27 1.27)) hide)
     )
+    (property "Digikey Part  Number" "YAG2303CT-ND" (id 4) (at 215.9 218.44 0)
+      (effects (font (size 1.27 1.27)) hide)
+    )
     (pin "1")
     (pin "2")
@@
       (effects (font (size 1.27 1.27)) hide)
     )
+    (property "Digikey Part  Number" "n/a" (id 4) (at 133.35 114.3 0)
+      (effects (font (size 1.27 1.27)) hide)
+    )
     (pin "1")
   )
@@
     )
     (property "Datasheet" "http://www.winbond.com/resource-files/w25q128jv_dtr%20revc%2003272018%20plus.pdf" (id 3) (at 69.85 210.82 0)
+      (effects (font (size 1.27 1.27)) hide)
+    )
+    (property "Digikey Part  Number" "W25Q128JVSIMCT-ND" (id 4) (at 69.85 210.82 0)
       (effects (font (size 1.27 1.27)) hide)
     )
@@
       (effects (font (size 1.27 1.27)) hide)
     )
+    (property "Digikey Part  Number" "YAG2303CT-ND" (id 4) (at 208.28 220.98 0)
+      (effects (font (size 1.27 1.27)) hide)
+    )
     (pin "1")
     (pin "2")
@@
       (effects (font (size 1.27 1.27)) hide)
     )
+    (property "Digikey Part  Number" "311-22.0KLRCT-ND " (id 4) (at 351.79 185.42 0)
+      (effects (font (size 1.27 1.27)) hide)
+    )
     (pin "1")
     (pin "2")
@@
       (effects (font (size 1.27 1.27)) hide)
     )
+    (property "Digikey Part  Number" "311-10KJRCT-ND " (id 4) (at 104.14 237.49 0)
+      (effects (font (size 1.27 1.27)) hide)
+    )
     (pin "1")
     (pin "2")
@@
       (effects (font (size 1.27 1.27)) hide)
     )
+    (property "Digikey Part  Number" "YAG3085CT-ND" (id 4) (at 111.76 185.42 0)
+      (effects (font (size 1.27 1.27)) hide)
+    )
     (pin "1")
     (pin "2")
@@
     )
     (path "/4df2aa83-28ad-49a5-8d29-dea8b0eada16"
-      (reference "R10") (unit 1) (value "5") (footprint "Resistor_SMD:R_0402_1005Metric")
+      (reference "R10") (unit 1) (value "330") (footprint "Resistor_SMD:R_0402_1005Metric")
     )
     (path "/b41ccc53-152f-4898-8730-7b3768ac122f"
