File: Rp2040 wearable dev boards w wireless.kicad_pcb (KiCad board)
At the start: 4 copper layers, 40 x 65.7 mm, 79 parts, among them IC1 NRF24L01P-R7, J1 battery plug, J2 DX07S016JA1R1500, J3 Conn_01x20, J4 Conn_01x20, J6 EMPCB.SMAFSTJ.B.HT, Q1 Si2301, SW1 B3U-1100P, SW2 power Switch, U1 MCP73831T-4ADI/OT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

Commit message: finished
Changed lines of the file:
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@@
     (property "Sheetname" "")
     (attr smd)
-    (fp_text reference "R11" (at -0.153641 1.75) (layer "F.SilkS")
+    (fp_text reference "R11" (at -0.75 1.25) (layer "F.SilkS")
       (effects (font (size 1 1) (thickness 0.15)))
     )
